File: PCB/SatNOGS_Encoder/encoder_as5601/encoder_as5601.sch (KiCad schematic (older format))
At the start: 7 parts, among them P1 CONN_02X05, Q1 Q_NMOS_GSD, U1 AS5601

Commit message: wip
Connections:
- net SCL: now also P1.10 (P10); no longer P1.7 (P7)
- net SDA: now also P1.7 (P7); no longer P1.10 (P10)
Changed lines of the file:
@@
 	-1   0    0    1
 $EndComp
-Text Label 5110 4510 0    60   ~ 0
+Text Label 5110 4410 0    60   ~ 0
 SCL
-Text Label 5910 4410 2    60   ~ 0
+Text Label 5910 4510 2    60   ~ 0
 SDA
 $Comp
@@
 $EndComp
 Connection ~ 4860 4710
-Text Label 5110 4410 0    60   ~ 0
+Text Label 5910 4410 2    60   ~ 0
 SDA
-Text Label 5910 4510 2    60   ~ 0
+Text Label 5110 4510 0    60   ~ 0
 SCL
 $Comp
